File: BUCKY_POWER/BUCKY_POWER.kicad_sch (KiCad schematic)
At the start: 1 part

Commit message: Started POWER
Parts:
- added C? (x3): C, symbol Device:C_Small
- added D?: DS, symbol Device:D_Schottky_Small
- added D?: LED, symbol Device:LED
- added D?: Z, symbol Device:D_Zener_Small
- added F?: Fuse, symbol Device:Fuse
- added J?: BATT_2, symbol Connector_Generic:Conn_01x02
- added Q?: RV, symbol Device:Q_PMOS_GDS
- added Q?: UV/OVLO, symbol Device:Q_NMOS_GDS
- added Q?: OC, symbol Device:Q_NMOS_GDS
- added R? (x8): 10k, symbol Device:R_Small
- added R?: 120R, symbol Device:R_Small
- added R? (x2): 100k, symbol Device:R_Small
- added R? (x2): R, symbol Device:R_Small
- added R?: 270R, symbol Device:R_Small
- added R?: 1M, symbol Device:R_Small
- added U? (x3): LM393, symbol Comparator:LM393
- added U?: LM9061_M, Package_SO:SOIC-8_3.9x4.9mm_P1.27mm, symbol BUCKY_POWER:LM9061_M
- added U?: AND, symbol 74xGxx:74AHC1G08
- added U?: BTS724G, Package_SO:Infineon_PG-DSO-20-32, symbol Power_Management:BTS724G
- J?: value Conn_01x02 -> BATT_1
Connections:
- net +12V: now also U?.13 (OUT4), U?.14 (OUT3), U?.17 (OUT2), U?.18 (OUT1); no longer J?.1 (Pin_1)
- net -BATT: now also C?.2, C?.2, C?.2, D?.1 (K), J?.2 (Pin_2), R?.1, R?.1, R?.1, R?.2, R?.2, R?.2, U?.3 (GND), U?.3 (GND), U?.4 (V-)
- new net: R?.1, R?.2, U?.6 (_)
- new net: R?.1, R?.2, U?.3 (+)
- new net: D?.2 (A), R?.2, U?.2 (-), U?.5 (+)
- new net: R?.2, U?.2, U?.7
- new net: C?.1, U?.8 (DEL)
- new net: D?.1 (K), U?.5 (VCC), U?.7 (ON)
- new net: D?.1 (K), D?.2 (A), Q?.2 (D), Q?.3 (S), R?.1, R?.1
- new net: R?.2, U?.2 (THR)
- new net: D?.2 (A), Q?.1 (G), R?.1
- new net: F?.1, Q?.2 (D), U?.8 (V+)
- new net: R?.2, U?.2 (GND1/2)
- new net: R?.2, U?.1 (SNS)
- new net: R?.1, U?.6 (IREF)
- new net: R?.1, U?.1, U?.1
- new net: Q?.1 (G), R?.1, U?.4
- new net: C?.1, C?.1, Q?.3 (S), R?.2, U?.1 (VBB), U?.10 (VBB), U?.11 (VBB), U?.12 (VBB), U?.15 (VBB), U?.16 (VBB), U?.19 (VBB), U?.20 (VBB)
- new net: R?.2, U?.6 (GND3/4)
- new net +BATT: F?.2, J?.1 (Pin_1), J?.1 (Pin_1)
- new net GATE: Q?.1 (G), U?.4 (OUT)
- new net IN: R?.1, R?.1, U?.3 (IN1), U?.5 (IN2), U?.7 (IN3), U?.9 (IN4)
- new net IN_CONN: R?.2
- new net ST1: U?.4 (ST1/2), U?.8 (ST3/4)
- new net VCC: Q?.2 (D), Q?.3 (S), R?.1, R?.1, R?.2, R?.2, U?.5 (VCC)
Other:
- moved on the sheet: J?

Commit message: Power Done
Parts:
- removed C?: C, symbol Device:C_Small
- removed D?: DS, symbol Device:D_Schottky_Small
- removed D?: LED, symbol Device:LED
- removed Q?: UV/OVLO, symbol Device:Q_NMOS_GDS
- removed Q?: OC, symbol Device:Q_NMOS_GDS
- removed R?: 120R, symbol Device:R_Small
- removed R? (x3): 10k, symbol Device:R_Small
- removed R? (x2): R, symbol Device:R_Small
- removed U?: LM9061_M, Package_SO:SOIC-8_3.9x4.9mm_P1.27mm, symbol BUCKY_POWER:LM9061_M
- removed U?: AND, symbol 74xGxx:74AHC1G08
- added J?: 5V BUCK, symbol Connector_Generic:Conn_02x06_Odd_Even
- added Q?: RV, symbol Device:Q_PMOS_GDS
- added R?: 68k, symbol Device:R_Small
- added R?: 1k, symbol Device:R_Small
- added R?: 10k, symbol Device:R_Small
- added U?: NAND, symbol 74xGxx:74AHC1G00
- added U?: TL431DBZ, Package_TO_SOT_SMD:SOT-23, symbol Reference_Voltage:TL431DBZ
- added U?: TPS2592xx, Package_SON:VSON-10-1EP_3x3mm_P0.5mm_EP1.65x2.4mm_ThermalVias, symbol Power_Management:TPS2592xx
- R?: value 10k -> 20k
- R?: value 10k -> 75k
Connections:
- net -BATT: now also R?.1, R?.2, U?.2 (GND1/2), U?.6 (GND3/4), J?.3 (Pin_3), J?.4 (Pin_4), J?.5 (Pin_5), J?.6 (Pin_6), U?.11 (GND), U?.3 (A), U?.3 (GND); no longer R?.1, R?.2, R?.2
- net IN: now also R?.2; no longer R?.1
- net VCC: now also D?.1 (K), Q?.3 (S), R?.1, R?.1, U?.8 (V+), Q?.3 (S), R?.2, U?.5 (VCC); no longer R?.2
- net at U?.2 (-), U?.5 (+): now also R?.1, U?.1 (K), U?.2 (REF)
- net at R?.2, U?.7: now also U?.2
- net at D?.2 (A), Q?.1 (G): now also R?.2; no longer R?.1
- net at F?.1, Q?.2 (D): no longer U?.8 (V+)
- net at R?.1, U?.1: now also U?.1
- net at C?.1, C?.1, U?.1 (VBB)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: now also R?.1, Q?.2 (D), R?.1, R?.2, U?.3 (VIN), U?.4 (VIN), U?.5 (VIN); no longer R?.2
- new net: R?.1, R?.2, U?.6 (_)
- new net: R?.1, R?.2, U?.3 (+)
- new net: R?.2, U?.10 (ILIM)
- new net: Q?.1 (G), R?.2, U?.4
- new net: R?.1, U?.2 (EN/UVLO)
- new net +5V: J?.1 (Pin_1), J?.2 (Pin_2)
- new net EN: J?.11 (Pin_11)
- new net OUT: J?.7 (Pin_7), J?.8 (Pin_8), U?.6 (OUT), U?.7 (OUT), U?.8 (OUT)
- new net PG: J?.12 (Pin_12)
- no-connect marks 0 -> 3
Other:
- moved on the sheet: C?, J?, R?, U?, U?A, U?B, U?C

Commit message: Started Power pcb
Parts:
- removed R?: 270R, symbol Device:R_Small
- removed R?: 10k, symbol Device:R_Small
- removed U?: BTS724G, Package_SO:Infineon_PG-DSO-20-32, symbol Power_Management:BTS724G
- added C3: 100n, Capacitor_SMD:C_0805_2012Metric_Pad1.18x1.45mm_HandSolder, symbol Device:C_Small
- added C4: 10n, Capacitor_SMD:C_0805_2012Metric_Pad1.18x1.45mm_HandSolder, symbol Device:C_Small
- added J4: 12V, Connector_PinHeader_2.54mm:PinHeader_2x06_P2.54mm_Vertical, symbol Connector_Generic:Conn_02x06_Counter_Clockwise
- added J5: 5V, Connector_PinHeader_2.54mm:PinHeader_2x06_P2.54mm_Vertical, symbol Connector_Generic:Conn_02x06_Counter_Clockwise
- added J6: GND, Connector_PinHeader_2.54mm:PinHeader_2x06_P2.54mm_Vertical, symbol Connector_Generic:Conn_02x06_Counter_Clockwise
- added R10, R11, R12: 4.7k, Resistor_SMD:R_0805_2012Metric_Pad1.20x1.40mm_HandSolder, symbol Device:R_Small
- added R13: 1.2k, Resistor_SMD:R_0805_2012Metric_Pad1.20x1.40mm_HandSolder, symbol Device:R_Small
- added R15: 47R, Resistor_SMD:R_0805_2012Metric_Pad1.20x1.40mm_HandSolder, symbol Device:R_Small
- added U5: BTS7004-1EPP, Package_SO:Infineon_PG-TSDSO-14-22, symbol Power_Management:BTS7004-1EPP
- C1: renamed from C?; value C -> 1u; footprint (none) -> Capacitor_SMD:C_1206_3216Metric_Pad1.33x1.80mm_HandSolder
- C2: renamed from C?; value C -> 100n; footprint (none) -> Capacitor_SMD:C_0805_2012Metric_Pad1.18x1.45mm_HandSolder
- D1: renamed from D?; footprint (none) -> Diode_SMD:D_SOD-123
- F1: renamed from F?; footprint (none) -> BUCKY_POWER:01530008
- J1, J2: renamed from J?; footprint (none) -> Connector_JST:JST_XH_B2B-XH-A_1x02_P2.50mm_Vertical
- J3: renamed from J?; footprint (none) -> Connector_PinSocket_2.54mm:PinSocket_2x06_P2.54mm_Vertical_SMD
- Q1, Q2: renamed from Q?; footprint (none) -> Package_TO_SOT_SMD:TO-252-2
- R1, R14, R2, R3, R4, R5, R6, R7, R8, R9: renamed from R?; footprint (none) -> Resistor_SMD:R_0805_2012Metric_Pad1.20x1.40mm_HandSolder
- U2: renamed from U?; value LM393 -> LM393BIDR; footprint (none) -> Package_SO:SOIC-8_3.9x4.9mm_P1.27mm
- U3: renamed from U?; value NAND -> CD40107BPSR; footprint (none) -> Package_SO:SOIC-8_3.9x4.9mm_P1.27mm
- gave numbers to parts that had none: 2
Connections:
- net +12V: now also C4.1, J4.1 (Pin_1), J4.10 (Pin_10), J4.11 (Pin_11), J4.12 (Pin_12), J4.2 (Pin_2), J4.3 (Pin_3), J4.4 (Pin_4), J4.5 (Pin_5), J4.6 (Pin_6), J4.7 (Pin_7), J4.8 (Pin_8), J4.9 (Pin_9), U5.10 (OUT), U5.12 (OUT), U5.13 (OUT), U5.14 (OUT), U5.8 (OUT), U5.9 (OUT)
- net +5V: now also J5.1 (Pin_1), J5.2 (Pin_2), J5.3 (Pin_3), J5.4 (Pin_4), J5.5 (Pin_5), J5.6 (Pin_6), J5.7 (Pin_7), J5.8 (Pin_8), J5.9 (Pin_9)
- net -BATT: now also C3.2, C4.2, J6.1 (Pin_1), J6.10 (Pin_10), J6.11 (Pin_11), J6.12 (Pin_12), J6.2 (Pin_2), J6.3 (Pin_3), J6.4 (Pin_4), J6.5 (Pin_5), J6.6 (Pin_6), J6.7 (Pin_7), J6.8 (Pin_8), J6.9 (Pin_9), R13.1, R15.1
- net IN: now also J5.12 (Pin_12), R11.2
- net ST1: now also J5.11 (Pin_11), R12.2
- net at C1.1, C2.1, Q2.2 (D)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: now also U5.15 (VS)
- new net: R10.2, R13.2, U5.4 (IS)
- new net: R15.2, U5.1 (GND)
- new net: R11.1, U5.2 (IN)
- new net: R12.1, U5.3 (DEN)
- new net IS: C3.1, J5.10 (Pin_10), R10.1
Other:
- moved on the sheet: C1, C2

Commit message: Updates to PCB POWER
Parts:
- added C5, C6: 100u, Capacitor_SMD:CP_Elec_6.3x7.7, symbol Device:C_Polarized_Small
- added D2: BATT, LED_SMD:LED_0805_2012Metric, symbol Device:LED
- added D3: UV, LED_SMD:LED_0805_2012Metric, symbol Device:LED
- added D4: 12V, LED_SMD:LED_0805_2012Metric, symbol Device:LED
- added D5: 5V, LED_SMD:LED_0805_2012Metric, symbol Device:LED
- added R16, R17, R19, R20, R21: 100k, Resistor_SMD:R_0805_2012Metric_Pad1.20x1.40mm_HandSolder, symbol Device:R_Small
- added R18: 10k, Resistor_SMD:R_0805_2012Metric_Pad1.20x1.40mm_HandSolder, symbol Device:R_Small
- added SW1: SW_MOTOR, BUCKY_POWER:EG1218, symbol Switch:SW_SPDT
- added SW2: SW_POWER, BUCKY_POWER:EG1218, symbol Switch:SW_SPDT
- added SW3: 5V_EN, BUCKY_POWER:EG1218, symbol Switch:SW_SPDT
- C1: value 1u -> 10u
- R9: value 10k -> 100k
Connections:
- net +12V: now also C5.1, C6.1, R20.2
- net +5V: now also R16.2, R21.2
- net -BATT: now also C5.2, C6.2, D2.1 (K), D3.1 (K), D4.1 (K), D5.1 (K), SW1.2 (B), SW3.3 (C)
- net EN: now also R9.1, U4.2 (EN/UVLO), SW3.2 (B); no longer J3.11 (Pin_11)
- net IN: now also R16.1, SW1.3 (C)
- net VCC: now also R17.2, R18.1
- net at C1.1, C2.1, Q2.2 (D)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: now also R19.2
- net NAND: now reaches R8.2, U3.4
- net NAND: now also SW2.3 (C); no longer Q2.1 (G)
- new net: D4.2 (A), R20.1
- new net: D2.2 (A), R17.1
- new net: R18.2, SW2.1 (A)
- new net: D5.2 (A), R21.1
- new net: D3.2 (A), R19.1
- new net GATE: Q2.1 (G), SW2.2 (B)
- no-connect marks 3 -> 6
Other:
- moved on the sheet: C4, D1, Q1, R1, R8
