File: BUCKY_POWER/BUCKY_POWER.kicad_pcb (KiCad board)
At the start: 2 copper layers, 82 x 39 mm, 34 parts, among them J1 BATT_1, J2 BATT_2, J3 5V BUCK, J4 12V, J5 5V, J6 GND, Q1 RV, Q2 RV, U1 TL431DBZ, U2 LM393BIDR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

Commit message: Almost finished Power PCB
Parts:
- moved R9 8.12 mm to (85.9, 101.6), turned to -90 degrees
- moved C2 5.95 mm to (97.3, 101.2)
- moved C1 5.50 mm to (94.9, 101.4)
- moved R14 4.48 mm to (92.6, 101.5)
- moved U2 0.15 mm to (63.8, 97.1)
Connections:
- U5 pad 11: unconnected-(U5-Pad11) -> +12V
Routing:
- net VCC: track 68.6 -> 27.3 mm
- net Net-(Q2-Pad1): track 13.0 -> 38.2 mm
- net /ST1: track 0.00 -> 21.9 mm, vias 0 -> 1
- net /IS: track 2.82 -> 24.5 mm
- net /IN: track 0.00 -> 20.3 mm, vias 0 -> 1
- net Net-(R6-Pad2): track 0.00 -> 19.8 mm, vias 0 -> 2
- net +BATT: track 17.1 -> 0.00 mm
- net -BATT: track 0.00 -> 11.2 mm, vias 0 -> 6
- net Net-(C1-Pad1): track 7.06 -> 15.0 mm, vias 0 -> 2
- net Net-(R9-Pad1): track 0.00 -> 6.07 mm
- net Net-(D1-Pad2): track 0.00 -> 6.03 mm
- net Net-(R7-Pad1): track 17.8 -> 23.1 mm, vias 0 -> 2
- net Net-(R14-Pad2): track 0.00 -> 2.55 mm, vias 0 -> 2
- net Net-(R4-Pad2): track 5.88 -> 8.05 mm
- added copper zone on F.Cu, net +12V
- added copper zone on F.Cu, net +5V
- added copper zone on F.Cu, net +BATT
- added copper zone on B.Cu, net -BATT
- added copper zone on F.Cu, net -BATT
- added copper zone on F.Cu, net /OUT
- added copper zone on F.Cu, net Net-(C1-Pad1)
- added copper zone on F.Cu, net Net-(F1-Pad1)
- added copper zone on F.Cu, net VCC

Commit message: Finished POWER
Parts:
- moved C4 55.0 mm to (148.0, 65.5), turned to 0 degrees
- moved C2 53.1 mm to (134.9, 63.7)
- moved 12V_CONN 53.0 mm to (147.9, 62.5)
- moved 5V_CONN 53.0 mm to (133.5, 80.4)
- moved BATT_1 53.0 mm to (76.8, 52.5)
- moved BATT_2 53.0 mm to (76.8, 61.5)
- moved BUCK 53.0 mm to (127.1, 71.1)
- moved C1 53.0 mm to (132.4, 63.9)
- moved C3 53.0 mm to (117.0, 65.3)
- moved D1 53.0 mm to (95.8, 57.0)
- moved F1 53.0 mm to (84.3, 57.4)
- moved Q1 53.0 mm to (93.0, 50.0)
- moved Q2 53.0 mm to (126.7, 50.0)
- moved R1 53.0 mm to (91.2, 57.0)
- moved R10 53.0 mm to (120.3, 63.0)
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- renumbered J4 to 12V_CONN, J5 to 5V_CONN, J2 to BATT_1, J1 to BATT_2, J3 to BUCK, J6 to GND_CONN
Other:
- board text added: "+"
- board text added: "-"
- board text added: "Power Protection Board By Pixeljoch 01-2023"
- board text added: "mom I swear this won't catch fire."

Commit message: Updates to PCB POWER
Parts:
- added C5: 100u, Capacitor_SMD:CP_Elec_6.3x7.7, F.Cu at (97.8, 92.2)
- added C6: 100u, Capacitor_SMD:CP_Elec_6.3x7.7, F.Cu at (105.3, 92.2)
- added D2: BATT, LED_SMD:LED_0805_2012Metric, F.Cu at (52.7, 102.8)
- added D3: UV, LED_SMD:LED_0805_2012Metric, F.Cu at (83.8, 91.0)
- added D4: 12V, LED_SMD:LED_0805_2012Metric, F.Cu at (101.8, 101.0)
- added D5: 5V, LED_SMD:LED_0805_2012Metric, F.Cu at (104.3, 109.5)
- added R16: 100k, Resistor_SMD:R_0805_2012Metric_Pad1.20x1.40mm_HandSolder, F.Cu at (80.1, 116.4)
- added R17: 100k, Resistor_SMD:R_0805_2012Metric_Pad1.20x1.40mm_HandSolder, F.Cu at (52.8, 98.5)
- added R18: 10k, Resistor_SMD:R_0805_2012Metric_Pad1.20x1.40mm_HandSolder, F.Cu at (72.2, 92.0)
- added R19: 100k, Resistor_SMD:R_0805_2012Metric_Pad1.20x1.40mm_HandSolder, F.Cu at (84.6, 88.1)
- added R20: 100k, Resistor_SMD:R_0805_2012Metric_Pad1.20x1.40mm_HandSolder, F.Cu at (103.9, 101.0)
- added R21: 100k, Resistor_SMD:R_0805_2012Metric_Pad1.20x1.40mm_HandSolder, F.Cu at (104.3, 105.8)
- added SW1: SW_MOTOR, BUCKY_POWER:EG1218, F.Cu at (76.2, 112.5)
- added SW2: SW_POWER, BUCKY_POWER:EG1218, F.Cu at (69.5, 87.8)
- added SW3: 5V_EN, BUCKY_POWER:EG1218, F.Cu at (101.0, 112.5)
- C1: value 1u -> 10u
- R9: value 10k -> 100k
- moved C4 55.0 mm to (106.0, 101.0), turned to -90 degrees
- moved C2 53.1 mm to (97.3, 101.2)
- moved C1 53.0 mm to (94.9, 101.4)
- moved C3 53.0 mm to (79.5, 102.8)
- moved D1 53.0 mm to (58.3, 94.5)
- moved F1 53.0 mm to (46.8, 94.9)
- moved J1 53.0 mm to (39.3, 99.0)
- moved J2 53.0 mm to (39.3, 90.0)
- moved J3 53.0 mm to (89.6, 108.6)
- moved J4 53.0 mm to (110.4, 100.0)
- moved J5 53.0 mm to (96.0, 117.9)
- moved Q1 53.0 mm to (55.5, 87.5)
- moved Q2 53.0 mm to (89.2, 87.5)
- moved R1 53.0 mm to (53.8, 94.5)
- moved R10 53.0 mm to (82.8, 100.5)
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- renumbered BATT_2 to J1, BATT_1 to J2, BUCK to J3, 12V_CONN to J4, 5V_CONN to J5, GND_CONN to J6
Connections:
- J3 pad 11: /EN -> unconnected-(J3-Pad11)
- Q2 pad 1: Net-(Q2-Pad1) -> /GATE
- R8 pad 2: Net-(Q2-Pad1) -> /NAND
- R9 pad 1: Net-(R9-Pad1) -> /EN
- U3 pad 4: Net-(Q2-Pad1) -> /NAND
- U4 pad 2: Net-(R9-Pad1) -> /EN
- U5 pad 11: +12V -> unconnected-(U5-Pad11)
Routing:
- net /NAND: track 0.00 -> 38.2 mm
- net Net-(Q2-Pad1): track 38.2 -> 0.00 mm
- net /EN: track 0.00 -> 26.9 mm, vias 0 -> 1
- net /IN: track 20.3 -> 34.1 mm
- net -BATT: track 11.2 -> 17.9 mm, vias 6 -> 9
- net Net-(R9-Pad1): track 6.07 -> 0.00 mm
- net Net-(D2-Pad2): track 0.00 -> 4.27 mm
- net +5V: track 0.00 -> 3.15 mm
- net VCC: track 27.3 -> 29.3 mm
- net Net-(D5-Pad2): track 0.00 -> 1.66 mm
- net /IS: track 24.5 -> 23.2 mm
Other:
- board text removed: "+"
- board text removed: "-"
- board text removed: "Power Protection Board By Pixeljoch 01-2023"
- board text removed: "mom I swear this won't catch fire."

Commit message: POWER Board mag de tyfus krijgen met al die reference designators
Parts:
- renumbered SW1 to 12V, J1 to BATT_1, J2 to BATT_2, SW2 to PWR
Connections:
- J5 pad 10: /IS -> +5V
- J5 pad 11: /ST1 -> /IS
- J5 pad 12: /IN -> /ST1
Routing:
- net /GATE: track 0.00 -> 22.8 mm
- net /NAND: track 38.2 -> 30.3 mm
- net /IN: track 34.1 -> 28.3 mm
- net Net-(R18-Pad2): track 0.00 -> 5.52 mm
- net /ST1: track 21.9 -> 19.3 mm
- net Net-(D4-Pad2): track 0.00 -> 2.11 mm
- net Net-(D3-Pad2): track 0.00 -> 1.98 mm
- net /IS: track 23.2 -> 21.9 mm
- net -BATT: track 17.9 -> 19.0 mm, vias 9 -> 10
Other:
- board text added: "+"
- board text added: "-"
- board text added: "OFF"
- board text added: "ON"

Commit message: Finished PCBS
Parts:
- added REF**: KiCad-Logo2_5mm_SilkScreen, Symbol:KiCad-Logo2_5mm_SilkScreen, B.Cu at (101.4, 84.4)
- added REF**: OSHW-Logo2_7.3x6mm_SilkScreen, Symbol:OSHW-Logo2_7.3x6mm_SilkScreen, B.Cu at (89.2, 84.8)
- 12V CONN: renamed from J4
- 5V BUCK: renamed from J3
- 5V CONN: renamed from J5
- GND CONN: renamed from J6
- moved C3 0.50 mm to (79.5, 103.3)
- moved R9 0.30 mm to (85.9, 101.9)
- moved C2 0.10 mm to (97.3, 101.1)
- renumbered SW3 to ON
Routing:
- net -BATT: track 19.0 -> 18.5 mm
Other:
- board text added: "5V"
- board text added: "BUCKY POWER PROTECTION BOARD DESIGNED BY PIXELJOCH 01-2023 V-1.0"
- board text added: "Mom i swear"
- board text added: "TEAM BUCKY"
- board text added: "it wont catch fire"
