File: BUCKY_IR/BUCKY_IR.kicad_pcb (KiCad board)
At the start: 2 copper layers, 189.9 x 157.6 mm, 28 parts, among them J1 SERIAL_CONN, J2 CAN_CONN_UP, J3 CAN_CONN_DOWN, U1 TSSP96038TR, U10 TSSP96038TR, U11 TSSP96038TR, U12 TSSP96038TR, U13 TSSP96038TR, U14 TSSP96038TR, U15 TSSP96038TR, U16 TSSP96038TR, U17 TSSP96038TR, U18 ESP32-WROOM-32D, U2 TSSP96038TR, U3 TSSP96038TR, U4 TSSP96038TR, U5 SN65HVD230, U6 TSSP96038TR, U7 TSSP96038TR, U8 TSSP96038TR, U9 TSSP96038TR

Commit message: Some IR changes
Parts:
- removed the U17 at (270.4, 63.3)
- added U19: AMS1117, Package_TO_SOT_SMD:SOT-223-3_TabPin2, F.Cu at (96.9, 44.6)
- added U5: TSSP96038TR, BUCKY_IR:TSSP96038, F.Cu at (213.1, 81.5)
- moved U13 229.7 mm to (30.5, 81.5), turned to -90 degrees
- moved U11 222.5 mm to (57.2, 146.1), turned to -45 degrees
- moved U12 219.3 mm to (37.4, 116.4), turned to -67.5 degrees
- moved U14 218.4 mm to (37.4, 46.6), turned to -112.5 degrees
- moved U15 210.4 mm to (49.2, 23.4), turned to -130 degrees
- moved U10 208.5 mm to (86.9, 165.9), turned to -22.5 degrees
- moved U9 191.3 mm to (121.8, 172.8)
- moved U16 186.9 mm to (86.9, 23.5), turned to 180 degrees
- moved U1 146.1 mm to (121.8, 23.5), turned to 180 degrees
- moved U7 133.3 mm to (186.4, 146.1), turned to 45 degrees
- moved U2 127.4 mm to (156.7, 23.5), turned to 180 degrees
- moved U8 123.1 mm to (156.7, 165.9), turned to 22.5 degrees
- moved U3 96.1 mm to (194.4, 23.4), turned to 130 degrees
- moved U6 85.3 mm to (206.2, 116.4), turned to 67.5 degrees
- moved U4 50.2 mm to (206.2, 46.6), turned to 112.5 degrees
- renumbered U5 to U17
Connections:
- U10 pad 4: /IR_3 -> /IR_10
- U11 pad 4: /IR_7 -> /IR_11
- U12 pad 4: /IR_11 -> /IR_12
- U13 pad 4: /IR_15 -> /IR_13
- U14 pad 4: /IR_4 -> /IR_14
- U15 pad 4: /IR_8 -> /IR_15
- U16 pad 4: /IR_12 -> /IR_16
- U2 pad 4: /IR_5 -> /IR_2
- U3 pad 4: /IR_9 -> /IR_3
- U4 pad 4: /IR_13 -> /IR_4
- U6 pad 4: /IR_2 -> /IR_6
- U7 pad 4: /IR_6 -> /IR_7
- U8 pad 4: /IR_10 -> /IR_8
- U9 pad 4: /IR_14 -> /IR_9

Commit message: More IR dev
Parts:
- added C4: 10u, Capacitor_SMD:CP_Elec_6.3x7.7, F.Cu at (105.4, 47.6)
- added C5: 100n, Capacitor_SMD:C_0805_2012Metric_Pad1.18x1.45mm_HandSolder, F.Cu at (104.9, 42.9)
- J1, J2, J3: footprint Connector_JST:JST_PH_B6B-PH-K_1x06_P2.00mm_Vertical -> Connector_JST:JST_PH_S6B-PH-SM4-TB_1x06-1MP_P2.00mm_Horizontal
- U18: value ESP32-WROOM-32D -> ESP32-WROOM-32U; footprint RF_Module:ESP32-WROOM-32 -> RF_Module:ESP32-WROOM-32U
- U19: value AMS1117 -> AMS1117-5.0
- moved C3 22.5 mm to (176.0, 83.5)
- moved D1 22.5 mm to (181.9, 92.3)
- moved R3 22.5 mm to (181.8, 97.8)
- moved R2 22.5 mm to (180.9, 86.1)
- moved U17 17.0 mm to (96.6, 36.3), turned to 180 degrees
- moved C2 7.38 mm to (83.8, 40.3)
- moved J1 7.31 mm to (141.0, 57.7)
- moved C1 7.21 mm to (83.8, 47.6)
- moved R1 4.21 mm to (89.0, 36.2), turned to 90 degrees
- moved U19 3.86 mm to (94.9, 47.9), turned to 90 degrees
- moved J3 2.62 mm to (86.1, 57.7)
- moved J2 1.89 mm to (103.5, 57.7)
- moved U18 1.15 mm to (122.1, 44.1), turned to 180 degrees
Connections:
- C1 pad 1: +3V3 -> +5V
- C2 pad 1: +3V3 -> +5V
- C3 pad 1: +3V3 -> +5V
- J2 pad 1: +3V3 -> +5V
- J2 pad 2: /CAN_H -> +5V
- J2 pad 3: /CAN_L -> +3V3
- J2 pad 4: GND -> /CAN_H
- J2 pad 5: (no net) -> /CAN_L
- J2 pad 6: (no net) -> GND
- J3 pad 1: +3V3 -> +5V
- J3 pad 2: /CAN_H -> +5V
- J3 pad 3: /CAN_L -> +3V3
- J3 pad 4: GND -> /CAN_H
- J3 pad 5: (no net) -> /CAN_L
- J3 pad 6: (no net) -> GND
- U18 pad 10: /IR_10 -> /IR_4
- U18 pad 11: /IR_11 -> /IR_3
- U18 pad 12: /IR_12 -> /IR_2
- U18 pad 23: /IR_2 -> /IR_16
- U18 pad 27: /IR_3 -> /IR_15
- U18 pad 28: /IR_4 -> /IR_14
- U18 pad 30: /IR_5 -> /IR_13
- U18 pad 31: /IR_6 -> /IR_12
- U18 pad 33: /IR_7 -> /IR_11
- U18 pad 36: /IR_8 -> /IR_10
- U18 pad 6: /IR_15 -> /IR_8
- U18 pad 7: /IR_16 -> /IR_7
- U18 pad 8: /IR_13 -> /IR_6
- U18 pad 9: /IR_14 -> /IR_5
- U19 pad 1: unconnected-(U19-Pad1) -> GND
- U19 pad 2: unconnected-(U19-Pad2) -> +3V3
- U19 pad 3: unconnected-(U19-Pad3) -> +5V
Routing:
- net /IR_9: track 0.00 -> 219.2 mm, vias 0 -> 2
- net /IR_8: track 0.00 -> 215.0 mm
- net /IR_10: track 0.00 -> 191.7 mm, vias 0 -> 2
- net /IR_7: track 0.00 -> 183.0 mm
- net /IR_11: track 0.00 -> 162.4 mm, vias 0 -> 2
- net /IR_6: track 0.00 -> 145.7 mm
- net /IR_12: track 0.00 -> 130.6 mm, vias 0 -> 2
- net /IR_5: track 0.00 -> 111.0 mm
- net /IR_13: track 0.00 -> 106.3 mm, vias 0 -> 2
- net /IR_14: track 0.00 -> 82.5 mm, vias 0 -> 2
- net /IR_15: track 0.00 -> 76.5 mm, vias 0 -> 2
- net /IR_4: track 0.00 -> 76.4 mm
- net /IR_3: track 0.00 -> 72.6 mm
- net /IR_16: track 0.00 -> 39.8 mm, vias 0 -> 2
- net /IR_2: track 0.00 -> 33.1 mm
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
Commit message: Even more IR dev
Parts:
- C1: value 470u -> 100u
- moved C2 13.0 mm to (94.5, 47.7), turned to -90 degrees
- moved R1 11.1 mm to (97.6, 43.3)
- moved U19 10.7 mm to (89.3, 38.8), turned to 0 degrees
- moved C5 9.03 mm to (104.2, 33.9)
- moved U17 6.62 mm to (102.6, 39.1)
- moved C4 2.30 mm to (103.1, 47.7), turned to -90 degrees
- moved C1 2.30 mm to (86.1, 47.6), turned to -90 degrees
Routing:
- net +3V3: track 0.00 -> 687.2 mm
- net +5V: track 0.00 -> 64.1 mm
- net /TX: track 0.00 -> 34.7 mm
- net /RX: track 0.00 -> 32.7 mm
- net /CAN_H: track 0.00 -> 31.9 mm, vias 0 -> 2
- net /CAN_L: track 0.00 -> 26.8 mm, vias 0 -> 2
- net /IR_10: track 191.7 -> 203.9 mm
- net /IR_9: track 219.2 -> 231.3 mm
- net /IR_11: track 162.4 -> 174.3 mm
- net /CAN_TX: track 0.00 -> 8.54 mm
- net /CAN_RX: track 0.00 -> 8.54 mm
- net /IR_12: track 130.6 -> 138.8 mm
- net /IR_2: track 33.1 -> 40.6 mm
- net /IR_13: track 106.3 -> 113.7 mm
- net /IR_15: track 76.5 -> 72.2 mm
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
Commit message: Finished IR PCB
Parts:
- removed C2: 10u, Capacitor_SMD:CP_Elec_6.3x7.7
- added C3: 10u, Capacitor_SMD:CP_Elec_6.3x7.7, F.Cu at (70.5, 47.6)
- moved C3 111.5 mm to (68.3, 54.9), turned to -90 degrees
- moved D1 69.7 mm to (139.0, 37.4)
- moved R2 66.2 mm to (139.0, 34.9)
- moved R3 64.4 mm to (137.1, 51.5), turned to 180 degrees
- moved C5 15.3 mm to (97.3, 47.6), turned to -90 degrees
- moved C1 8.30 mm to (77.8, 47.6), turned to 90 degrees
- moved U19 8.00 mm to (87.5, 46.6)
- moved J3 7.86 mm to (78.2, 57.6)
- moved R1 3.55 mm to (94.1, 43.9), turned to 0 degrees
- moved U17 2.30 mm to (104.9, 39.1)
- moved C4 1.17 mm to (102.0, 47.3), turned to 90 degrees
- moved J2 0.51 mm to (103.0, 57.6)
Routing:
- net +3V3: track 687.2 -> 787.4 mm, vias 0 -> 2
- net +5V: track 64.1 -> 126.0 mm
- net /IO_0: track 0.00 -> 59.7 mm, vias 0 -> 2
- net /CAN_H: track 31.9 -> 59.8 mm
- net /CAN_L: track 26.8 -> 53.1 mm
- net Net-(J1-Pad2): track 0.00 -> 12.3 mm
- net /LED: track 0.00 -> 11.5 mm, vias 0 -> 2
- net Net-(D1-Pad2): track 0.00 -> 2.51 mm
- net /CAN_TX: track 8.54 -> 6.24 mm
- net /CAN_RX: track 8.54 -> 6.24 mm
- net /RX: track 32.7 -> 34.7 mm
- net /TX: track 34.7 -> 35.8 mm
- net GND: vias 0 -> 25
- added copper zone on B.Cu, net GND
- added copper zone on F.Cu, net GND

Commit message: Some LIGHT dev
Routing:
- net +3V3: track 787.4 -> 788.9 mm

Commit message: Finished PCBS
Parts:
- added LED: LED, Connector_PinHeader_2.54mm:PinHeader_1x02_P2.54mm_Horizontal, F.Cu at (116.7, 61.4)
- added PD: PHOTODIODE, Connector_PinHeader_2.54mm:PinHeader_1x02_P2.54mm_Horizontal, F.Cu at (127.5, 61.7)
- added R4: 10k, Resistor_SMD:R_0805_2012Metric_Pad1.20x1.40mm_HandSolder, F.Cu at (130.4, 60.9)
- added R5: 120R, Resistor_SMD:R_0805_2012Metric_Pad1.20x1.40mm_HandSolder, F.Cu at (120.5, 61.6)
- added REF**: KiCad-Logo2_5mm_SilkScreen, Symbol:KiCad-Logo2_5mm_SilkScreen, F.Cu at (157.4, 59.4)
- added REF**: OSHW-Logo2_7.3x6mm_SilkScreen, Symbol:OSHW-Logo2_7.3x6mm_SilkScreen, F.Cu at (170.0, 59.8)
- C1: value 100u -> 470u
- renumbered C3 to C2
Connections:
- U18 pad 14: unconnected-(U18-Pad14) -> /PD
Routing:
- net /PD: track 0.00 -> 30.9 mm, vias 0 -> 1
- net /IR_9: track 231.3 -> 239.4 mm
- net /IR_12: track 138.8 -> 146.5 mm
- net /IR_11: track 174.3 -> 177.7 mm
- net +3V3: track 788.9 -> 792.2 mm
- net Net-(J5-Pad1): track 0.00 -> 2.92 mm
- net /IR_13: track 113.7 -> 112.2 mm
- net /IR_10: track 203.9 -> 205.1 mm
Other:
- outline, holes or cut-outs redrawn
- board text added: "(nu ook in infrarood)"
- board text added: "BUCKY PULSED IR BOARD DESIGNED BY PIXELJOCH 01-2023 V-2.0"
- board text added: "TEAM BUCKY"
- board text added: "ik zie alles"

Commit message: chore: start on schematics
Parts:
- removed D1: LED, LED_SMD:LED_0805_2012Metric_Pad1.15x1.40mm_HandSolder
- removed the J1 at (141.0, 57.7)
- removed LED: LED, Connector_PinHeader_2.54mm:PinHeader_1x02_P2.54mm_Horizontal
- removed PD: PHOTODIODE, Connector_PinHeader_2.54mm:PinHeader_1x02_P2.54mm_Horizontal
- removed R2, R5: 120R, Resistor_SMD:R_0805_2012Metric_Pad1.20x1.40mm_HandSolder
- removed R3, R4: 10k, Resistor_SMD:R_0805_2012Metric_Pad1.20x1.40mm_HandSolder
- removed REF**: KiCad-Logo2_5mm_SilkScreen, Symbol:KiCad-Logo2_5mm_SilkScreen
- removed REF**: OSHW-Logo2_7.3x6mm_SilkScreen, Symbol:OSHW-Logo2_7.3x6mm_SilkScreen
- removed U10, U11, U12, U13, U14, U15, U16, U2, U4, U5, U6: TSSP96038TR, BUCKY_IR:TSSP96038
- removed the U18 at (122.1, 44.1)
- removed the U7 at (186.4, 146.1)
- removed the U8 at (156.7, 165.9)
- added U20: TSSP96038TR, BUCKY_IR:TSSP96038, F.Cu at (82.3, 164.4)
- added U22: TSSP96038TR, BUCKY_IR:TSSP96038, F.Cu at (158.9, 164.4)
- added U23: TSSP96038TR, BUCKY_IR:TSSP96038, F.Cu at (187.0, 136.3)
- added U24: TSSP96038TR, BUCKY_IR:TSSP96038, F.Cu at (197.4, 98.0)
- added U25: TSSP96038TR, BUCKY_IR:TSSP96038, F.Cu at (187.0, 59.7)
- added U26: TSSP96038TR, BUCKY_IR:TSSP96038, F.Cu at (159.0, 31.7)
- added U27: TSSP96038TR, BUCKY_IR:TSSP96038, F.Cu at (120.7, 21.4)
- added U28: TSSP96038TR, BUCKY_IR:TSSP96038, F.Cu at (82.3, 31.6)
- added U29: TSSP96038TR, BUCKY_IR:TSSP96038, F.Cu at (54.4, 59.7)
- moved U3 180.0 mm to (54.3, 136.3), turned to -60 degrees
- moved U1 107.8 mm to (43.9, 98.0), turned to -90 degrees
- moved U18 2.18 mm to (120.6, 174.6)
- renumbered C2 to C1, C3 to C2, C1 to C3, C5 to C4, C4 to C5, J3 to J1, U9 to U18, U19 to U7, U17 to U8
Connections:
- U3 pad 4: /IR_3 -> /IR_1
- U8 pad 8: unconnected-(U17-Pad8) -> GND
Routing:
- net +3V3: track 792.2 -> 92.7 mm, vias 2 -> 1
- net /IR_9: track 239.4 -> 17.0 mm, vias 2 -> 1
- net /IR_8: track 215.0 -> 0.00 mm
- net /IR_10: track 205.1 -> 0.00 mm, vias 2 -> 0
- net /IR_7: track 183.0 -> 0.00 mm
- net /IR_11: track 177.7 -> 6.53 mm, vias 2 -> 1
- net /IR_12: track 146.5 -> 0.00 mm, vias 2 -> 0
- net /IR_6: track 145.7 -> 0.00 mm
- net /IR_13: track 112.2 -> 0.00 mm, vias 2 -> 0
- net /IR_5: track 111.0 -> 0.00 mm
- net /IR_14: track 82.2 -> 0.00 mm, vias 2 -> 0
- net /IR_4: track 76.4 -> 0.00 mm
- net /IR_3: track 71.3 -> 0.00 mm
- net /IO_0: track 59.7 -> 0.00 mm, vias 2 -> 0
- net /IR_2: track 40.6 -> 0.00 mm
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Other:
- board size 189.9 x 157.6 mm -> 156.1 x 156.1 mm
- board text added: "BUCKY PULSED IR BOARD DESIGNED BY koen1711 12-2023 V-1.0"
- board text added: "they said i couldn't do it, i couldn't"
- board text removed: "(nu ook in infrarood)"
- board text removed: "BUCKY PULSED IR BOARD DESIGNED BY PIXELJOCH 01-2023 V-2.0"
- board text removed: "ik zie alles"
