File: BUCKY_MOTOR_DRIVER/BUCKY_MOTOR_DRIVER.kicad_sch (KiCad schematic)
At the start: 8 parts, among them J1 P_INPUTS, J2 INPUTS, J3 OUT, U1 IFX9201SG

Commit message: Finished up IR sch, Main, Started Power
Parts:
- removed J1: P_INPUTS, Connector_PinSocket_2.54mm:PinSocket_1x04_P2.54mm_Vertical, symbol Connector_Generic:Conn_01x04
- removed J2: INPUTS, Connector_PinSocket_2.54mm:PinSocket_1x04_P2.54mm_Vertical, symbol Connector_Generic:Conn_01x04
- removed J3: OUT, Connector_PinHeader_2.54mm:PinHeader_1x02_P2.54mm_Vertical, symbol Connector_Generic:Conn_01x02
Connections:
- net OUT_2: now reaches C4.1, U1.7 (OUT2)
- net OUT_1: now reaches C3.1, U1.5 (OUT1)
Changed lines of the file:
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@@
   (junction (at 85.09 71.755) (diameter 0) (color 0 0 0 0)
   )
+  (junction (at 81.915 59.055) (diameter 0) (color 0 0 0 0)
+  )
   (junction (at 125.73 78.74) (diameter 0) (color 0 0 0 0)
   )
@@
   (junction (at 109.855 74.93) (diameter 0) (color 0 0 0 0)
   )
-  (junction (at 70.485 71.755) (diameter 0) (color 0 0 0 0)
-  )
   (junction (at 95.25 78.74) (diameter 0) (color 0 0 0 0)
-  )
-  (junction (at 91.44 59.055) (diameter 0) (color 0 0 0 0)
   )
   (junction (at 98.425 71.755) (diameter 0) (color 0 0 0 0)
@@
     (stroke (width 0) (type default) (color 0 0 0 0))
   )
-  (wire (pts (xy 70.485 71.755) (xy 74.295 71.755))
+  (wire (pts (xy 81.915 54.61) (xy 81.915 59.055))
     (stroke (width 0) (type default) (color 0 0 0 0))
   )
@@
     (stroke (width 0) (type default) (color 0 0 0 0))
   )
-  (wire (pts (xy 113.665 48.895) (xy 91.44 48.895))
-    (stroke (width 0) (type default) (color 0 0 0 0))
-  )
   (wire (pts (xy 109.855 74.295) (xy 109.855 74.93))
     (stroke (width 0) (type default) (color 0 0 0 0))
@@
     (stroke (width 0) (type default) (color 0 0 0 0))
   )
-  (wire (pts (xy 91.44 59.055) (xy 99.695 59.055))
-    (stroke (width 0) (type default) (color 0 0 0 0))
-  )
   (wire (pts (xy 66.675 64.135) (xy 70.485 64.135))
     (stroke (width 0) (type default) (color 0 0 0 0))
   )
-  (wire (pts (xy 66.675 71.755) (xy 70.485 71.755))
+  (wire (pts (xy 66.675 71.755) (xy 74.295 71.755))
     (stroke (width 0) (type default) (color 0 0 0 0))
   )
@@
     (stroke (width 0) (type default) (color 0 0 0 0))
   )
+  (wire (pts (xy 81.915 59.055) (xy 99.695 59.055))
+    (stroke (width 0) (type default) (color 0 0 0 0))
+  )
   (wire (pts (xy 70.485 56.515) (xy 70.485 64.135))
     (stroke (width 0) (type default) (color 0 0 0 0))
@@
     (stroke (width 0) (type default) (color 0 0 0 0))
   )
-  (wire (pts (xy 91.44 48.895) (xy 91.44 59.055))
-    (stroke (width 0) (type default) (color 0 0 0 0))
-  )
   (wire (pts (xy 120.015 64.135) (xy 134.62 64.135))
     (stroke (width 0) (type default) (color 0 0 0 0))
@@
     (stroke (width 0) (type default) (color 0 0 0 0))
   )
-  (wire (pts (xy 70.485 66.675) (xy 70.485 64.135))
-    (stroke (width 0) (type default) (color 0 0 0 0))
-  )
-  (wire (pts (xy 106.045 43.18) (xy 106.045 45.085))
-    (stroke (width 0) (type default) (color 0 0 0 0))
-  )
   (wire (pts (xy 95.25 78.74) (xy 95.25 80.645))
     (stroke (width 0) (type default) (color 0 0 0 0))
@@
     (stroke (width 0) (type default) (color 0 0 0 0))
   )
-  (wire (pts (xy 108.585 43.18) (xy 108.585 44.45))
-    (stroke (width 0) (type default) (color 0 0 0 0))
-  )
   (wire (pts (xy 98.425 71.755) (xy 98.425 74.93))
     (stroke (width 0) (type default) (color 0 0 0 0))
   )
-  (wire (pts (xy 66.675 69.215) (xy 70.485 69.215))
-    (stroke (width 0) (type default) (color 0 0 0 0))
-  )
-  (wire (pts (xy 113.665 43.18) (xy 113.665 48.895))
-    (stroke (width 0) (type default) (color 0 0 0 0))
-  )
-  (wire (pts (xy 111.125 43.18) (xy 111.125 45.085))
-    (stroke (width 0) (type default) (color 0 0 0 0))
-  )
   (wire (pts (xy 85.09 71.755) (xy 98.425 71.755))
     (stroke (width 0) (type default) (color 0 0 0 0))
   )
-  (wire (pts (xy 70.485 71.755) (xy 70.485 69.215))
-    (stroke (width 0) (type default) (color 0 0 0 0))
-  )
   (wire (pts (xy 125.73 88.265) (xy 125.73 90.17))
     (stroke (width 0) (type default) (color 0 0 0 0))
@@
     (stroke (width 0) (type default) (color 0 0 0 0))
   )
-  (wire (pts (xy 66.675 66.675) (xy 70.485 66.675))
-    (stroke (width 0) (type default) (color 0 0 0 0))
-  )
   (wire (pts (xy 120.015 56.515) (xy 121.285 56.515))
     (stroke (width 0) (type default) (color 0 0 0 0))
@@
     (stroke (width 0) (type default) (color 0 0 0 0))
   )
-  (wire (pts (xy 76.835 59.055) (xy 91.44 59.055))
+  (wire (pts (xy 76.835 59.055) (xy 81.915 59.055))
     (stroke (width 0) (type default) (color 0 0 0 0))
   )
@@
     (stroke (width 0) (type default) (color 0 0 0 0))
   )
-  (label "DIR" (at 106.045 45.085 270)
-    (effects (font (size 1.27 1.27)) (justify right bottom))
-  )
-  (label "PWM" (at 108.585 44.45 270)
-    (effects (font (size 1.27 1.27)) (justify right bottom))
-  )
-  (label "EN" (at 121.285 59.055 0)
-    (effects (font (size 1.27 1.27)) (justify left bottom))
-  )
-  (label "DIR" (at 99.06 56.515 180)
-    (effects (font (size 1.27 1.27)) (justify right bottom))
-  )
-  (label "PWM" (at 121.285 56.515 0)
-    (effects (font (size 1.27 1.27)) (justify left bottom))
-  )
-  (label "EN" (at 111.125 45.085 270)
-    (effects (font (size 1.27 1.27)) (justify right bottom))
-  )
-  (symbol (lib_id "Connector_Generic:Conn_01x02") (at 111.125 85.725 270) (unit 1)
-    (in_bom yes) (on_board yes) (fields_autoplaced)
-    (property "Reference" "J3" (id 0) (at 113.157 84.8903 90)
-      (effects (font (size 1.27 1.27)) (justify left))
-    )
-    (property "Value" "OUT" (id 1) (at 113.157 87.4272 90)
-      (effects (font (size 1.27 1.27)) (justify left))
-    )
-    (property "Footprint" "Connector_PinHeader_2.54mm:PinHeader_1x02_P2.54mm_Vertical" (id 2) (at 111.125 85.725 0)
-      (effects (font (size 1.27 1.27)) hide)
-    )
-    (property "Datasheet" "~" (id 3) (at 111.125 85.725 0)
-      (effects (font (size 1.27 1.27)) hide)
-    )
-    (pin "1")
-    (pin "2")
+  (hierarchical_label "GND" (shape bidirectional) (at 66.675 71.755 180)
+    (effects (font (size 1.27 1.27)) (justify right))
+  )
+  (hierarchical_label "DIR" (shape input) (at 99.06 56.515 180)
+    (effects (font (size 1.27 1.27)) (justify right))
+  )
+  (hierarchical_label "12V" (shape input) (at 66.675 64.135 180)
+    (effects (font (size 1.27 1.27)) (justify right))
+  )
+  (hierarchical_label "OUT_1" (shape output) (at 108.585 80.645 270)
+    (effects (font (size 1.27 1.27)) (justify right))
+  )
+  (hierarchical_label "OUT_2" (shape output) (at 111.125 80.645 270)
+    (effects (font (size 1.27 1.27)) (justify right))
+  )
+  (hierarchical_label "3V3" (shape input) (at 81.915 54.61 90)
+    (effects (font (size 1.27 1.27)) (justify left))
+  )
+  (hierarchical_label "PWM" (shape input) (at 121.285 56.515 0)
+    (effects (font (size 1.27 1.27)) (justify left))
+  )
+  (hierarchical_label "EN" (shape input) (at 121.285 59.055 0)
+    (effects (font (size 1.27 1.27)) (justify left))
   )
   (symbol (lib_id "BUCKY_MOTOR_DRIVER:IFX9201SG") (at 109.855 62.865 0) (unit 1)
@@
     (pin "9")
   )
-  (symbol (lib_id "Connector_Generic:Conn_01x04") (at 61.595 66.675 0) (mirror y) (unit 1)
-    (in_bom yes) (on_board yes) (fields_autoplaced)
-    (property "Reference" "J1" (id 0) (at 61.595 59.1652 0))
-    (property "Value" "P_INPUTS" (id 1) (at 61.595 61.7021 0))
-    (property "Footprint" "Connector_PinSocket_2.54mm:PinSocket_1x04_P2.54mm_Vertical" (id 2) (at 61.595 66.675 0)
-      (effects (font (size 1.27 1.27)) hide)
-    )
-    (property "Datasheet" "~" (id 3) (at 61.595 66.675 0)
-      (effects (font (size 1.27 1.27)) hide)
-    )
-    (pin "1")
-    (pin "2")
-    (pin "3")
-    (pin "4")
-  )
   (symbol (lib_id "power:GND") (at 109.855 75.565 0) (unit 1)
     (in_bom yes) (on_board yes) (fields_autoplaced)
@@
     (pin "2")
   )
-  (symbol (lib_id "Connector_Generic:Conn_01x04") (at 108.585 38.1 90) (unit 1)
-    (in_bom yes) (on_board yes) (fields_autoplaced)
-    (property "Reference" "J2" (id 0) (at 109.855 33.1302 90))
-    (property "Value" "INPUTS" (id 1) (at 109.855 35.6671 90))
-    (property "Footprint" "Connector_PinSocket_2.54mm:PinSocket_1x04_P2.54mm_Vertical" (id 2) (at 108.585 38.1 0)
-      (effects (font (size 1.27 1.27)) hide)
-    )
-    (property "Datasheet" "~" (id 3) (at 108.585 38.1 0)
-      (effects (font (size 1.27 1.27)) hide)
-    )
-    (pin "1")
-    (pin "2")
-    (pin "3")
-    (pin "4")
-  )
   (symbol (lib_id "Device:C") (at 85.09 67.945 0) (unit 1)

Commit message: Started POWER
Parts:
- C3, C4: value 33n -> 10n
Changed lines of the file:
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@@
       (effects (font (size 1.27 1.27)) (justify left))
     )
-    (property "Value" "33n" (id 1) (at 128.651 86.1572 0)
+    (property "Value" "10n" (id 1) (at 128.651 86.1572 0)
       (effects (font (size 1.27 1.27)) (justify left))
     )
@@
       (effects (font (size 1.27 1.27)) (justify left))
     )
-    (property "Value" "33n" (id 1) (at 98.171 86.1572 0)
+    (property "Value" "10n" (id 1) (at 98.171 86.1572 0)
       (effects (font (size 1.27 1.27)) (justify left))
     )
@@
     )
     (path "/b8e4c042-3cfb-471f-8ae0-2202a4ec8cc5"
-      (reference "C3") (unit 1) (value "33n") (footprint "Capacitor_SMD:C_0603_1608Metric_Pad1.08x0.95mm_HandSolder")
+      (reference "C3") (unit 1) (value "10n") (footprint "Capacitor_SMD:C_0603_1608Metric_Pad1.08x0.95mm_HandSolder")
     )
     (path "/5cbbabcd-2a05-4d4f-b19a-2e1b56abeaab"
-      (reference "C4") (unit 1) (value "33n") (footprint "Capacitor_SMD:C_0603_1608Metric_Pad1.08x0.95mm_HandSolder")
-    )
-    (path "/2f8c3cec-43a9-410d-ba41-e7cf91c88f62"
-      (reference "J1") (unit 1) (value "P_INPUTS") (footprint "Connector_PinSocket_2.54mm:PinSocket_1x04_P2.54mm_Vertical")
-    )
-    (path "/63479a35-1fbd-40f9-ac1b-e476935472f8"
-      (reference "J2") (unit 1) (value "INPUTS") (footprint "Connector_PinSocket_2.54mm:PinSocket_1x04_P2.54mm_Vertical")
-    )
-    (path "/0ff5c0a4-d8f6-4f10-b5b7-2fc797ee6059"
-      (reference "J3") (unit 1) (value "OUT") (footprint "Connector_PinHeader_2.54mm:PinHeader_1x02_P2.54mm_Vertical")
+      (reference "C4") (unit 1) (value "10n") (footprint "Capacitor_SMD:C_0603_1608Metric_Pad1.08x0.95mm_HandSolder")
     )
     (path "/142e849a-bfa2-47b1-88cc-63e1c177c828"

Commit message: chore: start on schematics
Connections:
- net +3V3 renamed +5V
Other:
- moved on the sheet: C1, C2, C3, C4, U1
