File: BUCKY_LIGHT/ANALOG_COMPARATOR_6_CHANNELS.kicad_sch (KiCad schematic)
At the start: 9 parts, among them IC1 LM319N_NOPB, IC2 LM319N_NOPB, IC3 LM319N_NOPB

Commit message: finish up robot (i think)
Parts:
- removed IC1, IC2, IC3: LM319N_NOPB, DIP794W56P254L1905H533Q14N, symbol ANALOG_COMP:LM319N_NOPB
- added IC6, IC7, IC8: LM319N_NOPB, BUCKY_LIGHT:ANALOG_COMP, symbol ANALOG_COMP:LM319N_NOPB
- LI10: renamed from LI1; footprint (none) -> LED_SMD:LED_PLCC-2_3.4x3.0mm_AK
- LI11: renamed from LI4; footprint (none) -> LED_SMD:LED_PLCC-2_3.4x3.0mm_AK
- LI12: renamed from LI3; footprint (none) -> LED_SMD:LED_PLCC-2_3.4x3.0mm_AK
- LI7: renamed from LI6; footprint (none) -> LED_SMD:LED_PLCC-2_3.4x3.0mm_AK
- LI8: renamed from LI2; footprint (none) -> LED_SMD:LED_PLCC-2_3.4x3.0mm_AK
- LI9: renamed from LI5; footprint (none) -> LED_SMD:LED_PLCC-2_3.4x3.0mm_AK
Connections:
- net +5V: now also IC6.11 (V+), IC7.11 (V+), IC8.11 (V+)
- net GND: now also IC6.3 (GND1), IC6.6 (V-), IC6.8 (GND2), IC7.3 (GND1), IC7.6 (V-), IC7.8 (GND2), IC8.3 (GND1), IC8.6 (V-), IC8.8 (GND2)
- net I1: now also IC7.4 (+INPUT1)
- net I2: now also IC7.9 (+INPUT2)
- net I3: now also IC8.4 (+INPUT1)
- net I4: now also IC8.9 (+INPUT2)
- net I5: now also IC6.4 (+INPUT1)
- net I6: now also IC6.9 (+INPUT2)
- net REF: now also IC6.10 (-INPUT2), IC6.5 (-INPUT1), IC7.10 (-INPUT2), IC7.5 (-INPUT1), IC8.10 (-INPUT2), IC8.5 (-INPUT1)
- net at LI10.2 (A): now also IC7.12 (OUTPUT1)
- net at LI12.2 (A): now also IC8.12 (OUTPUT1)
- net at LI8.2 (A): now also IC7.7 (OUTPUT2)
- net at LI9.2 (A): now also IC6.12 (OUTPUT1)
- net at LI7.2 (A): now also IC6.7 (OUTPUT2)
- net at LI11.2 (A): now also IC8.7 (OUTPUT2)
