File: BUCKY_MAIN/BUCKY_MAIN.kicad_pcb (KiCad board)
At the start: 4 copper layers, 156.4 x 156.4 mm, 41 parts, among them J1 Conn_01x10, J2 Conn_01x06, J4 Conn_01x06

Commit message: fix: BUCKY_MAIN v2?
Parts:
- removed D14: D, Diode_SMD:D_0805_2012Metric
- added D13: D, Diode_SMD:D_3220_8050Metric, F.Cu at (125.9, 153.7)
- added J3: Conn_01x01, Connector_PinHeader_2.54mm:PinHeader_1x01_P2.54mm_Vertical, F.Cu at (115.5, 66.6)
- A1: moved to F.Cu
- moved A1 14.1 mm to (110.4, 101.8)
- moved D7 12.7 mm to (131.8, 169.2)
- moved C12 7.05 mm to (102.1, 42.3), turned to 90 degrees
- moved J1 6.20 mm to (104.6, 139.2), turned to 0 degrees
- moved C6 5.96 mm to (159.6, 150.9), turned to 0 degrees
- moved C7 4.67 mm to (127.1, 169.2), turned to -90 degrees
- moved J2 4.42 mm to (153.6, 135.7)
- moved C11 4.30 mm to (69.7, 58.1)
- moved C1 3.61 mm to (115.0, 31.5), turned to 90 degrees
- moved D5 3.07 mm to (179.1, 131.8), turned to 0 degrees
- moved J4 2.97 mm to (118.7, 148.9), turned to 180 degrees
- moved C3 1.99 mm to (177.1, 65.6), turned to 0 degrees
- moved C5 1.50 mm to (177.4, 134.2), turned to 0 degrees
- moved C9 1.40 mm to (63.5, 134.2), turned to 180 degrees
- moved C4 1.02 mm to (187.2, 101.4), turned to 0 degrees
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Connections:
- A1 pad 0: unconnected-(A1-Pad0) -> /RX0
- A1 pad 1: unconnected-(A1-Pad1) -> /TX0
- A1 pad 10: unconnected-(A1-Pad10) -> /M3_PWM
- A1 pad 11: /IR_8 -> /IR_4
- A1 pad 12: /IR_9 -> /IR_6
- A1 pad 13: /IR_10 -> /IR_5
- A1 pad 17: /IR_6 -> /IR_9
- A1 pad 18: /SIG_RIGHT -> /SIG_LEFT
- A1 pad 19: /SIG_LEFT -> /SIG_RIGHT
- A1 pad 2: /M1_PWM -> /SIG_BACK
- A1 pad 20: /SIG_BACK -> /D20/SDA
- A1 pad 21: /SIG_FRONT -> /D21/SCL
- A1 pad 23: /IR_5 -> /D23
- A1 pad 25: unconnected-(A1-Pad25) -> /D25
- A1 pad 26: unconnected-(A1-Pad26) -> /D26
- A1 pad 27: unconnected-(A1-Pad27) -> /D27
- A1 pad 28: unconnected-(A1-Pad28) -> /D28
- A1 pad 29: unconnected-(A1-Pad29) -> /D29
- A1 pad 3: /M2_PWM -> /SIG_FRONT
- A1 pad 30: unconnected-(A1-Pad30) -> /D30
- A1 pad 31: unconnected-(A1-Pad31) -> /D31
- A1 pad 32: unconnected-(A1-Pad32) -> /D32
- A1 pad 33: unconnected-(A1-Pad33) -> /D33
- A1 pad 34: unconnected-(A1-Pad34) -> /D34
- A1 pad 35: unconnected-(A1-Pad35) -> /D35
- A1 pad 36: unconnected-(A1-Pad36) -> /D36
- A1 pad 37: unconnected-(A1-Pad37) -> /D37
- A1 pad 38: unconnected-(A1-Pad38) -> /D38
- A1 pad 39: unconnected-(A1-Pad39) -> /D39
- A1 pad 4: /M3_PWM -> /IR_7
- A1 pad 40: unconnected-(A1-Pad40) -> /D40
- A1 pad 41: unconnected-(A1-Pad41) -> /IR_10
- A1 pad 42: unconnected-(A1-Pad42) -> /D42
- A1 pad 43: /IR_4 -> /D43
- A1 pad 44: unconnected-(A1-Pad44) -> /D44
- A1 pad 45: unconnected-(A1-Pad45) -> /D45
- A1 pad 46: unconnected-(A1-Pad46) -> /D46
- A1 pad 47: unconnected-(A1-Pad47) -> /D47
- A1 pad 48: /IR_3 -> /D48
- A1 pad 49: unconnected-(A1-Pad49) -> /IR_11
- A1 pad 5: /IR_7 -> /IR_8
- A1 pad 51: /IR_2 -> /IR_12
- A1 pad 52: /IR_11 -> /IR_3
- A1 pad 53: /IR_12 -> /IR_2
- A1 pad 6: unconnected-(A1-Pad6) -> /D6
- A1 pad 7: unconnected-(A1-Pad7) -> /D7
- A1 pad 8: unconnected-(A1-Pad8) -> /M1_PWM
- A1 pad 9: unconnected-(A1-Pad9) -> /M2_PWM
- A1 pad AD10: unconnected-(A1-PadAD10) -> /A10
- A1 pad AD11: unconnected-(A1-PadAD11) -> /A11
- A1 pad AD12: unconnected-(A1-PadAD12) -> /A12
- A1 pad AD13: unconnected-(A1-PadAD13) -> /A13
- A1 pad AD14: unconnected-(A1-PadAD14) -> /A14
- A1 pad AD15: unconnected-(A1-PadAD15) -> /A15
- A1 pad AD4: unconnected-(A1-PadAD4) -> /A4
- A1 pad AD5: unconnected-(A1-PadAD5) -> /A5
- A1 pad AD6: unconnected-(A1-PadAD6) -> /A6
- A1 pad AD7: unconnected-(A1-PadAD7) -> /A7
- A1 pad AD8: unconnected-(A1-PadAD8) -> /A8
- A1 pad AD9: unconnected-(A1-PadAD9) -> /A9
- A1 pad AREF: +5V -> unconnected-(A1-PadAREF)
- A1 pad VIN: /VIN -> /VIN_12V
- D1 pad 2: +5V -> +3.3V
- D10 pad 2: +5V -> +3.3V
- D11 pad 2: +5V -> +3.3V
- D12 pad 2: +5V -> +3.3V
- D2 pad 2: +5V -> +3.3V
- D3 pad 2: +5V -> +3.3V
- D4 pad 2: +5V -> +3.3V
- D5 pad 2: +5V -> +3.3V
- D6 pad 2: +5V -> +3.3V
- D7 pad 2: +5V -> +3.3V
- D8 pad 2: +5V -> +3.3V
- D9 pad 2: +5V -> +3.3V
- J2 pad 1: Net-(D14-K) -> /VIN
Routing:
- net +3.3V: track 0.00 -> 458.8 mm, vias 0 -> 12
- net +5V: track 464.3 -> 25.1 mm, vias 11 -> 1
- net /VIN: track 166.2 -> 10.3 mm
- net /IR_3: track 40.2 -> 153.8 mm
- net /IR_11: track 139.9 -> 46.0 mm
- net /IR_2: track 55.9 -> 145.6 mm
- net /IR_4: track 33.9 -> 106.3 mm, vias 1 -> 0
- net /SIG_RIGHT: track 15.8 -> 71.7 mm
- net /SIG_LEFT: track 15.6 -> 71.2 mm
- net /IR_10: track 72.3 -> 26.2 mm
- net /SIG_BACK: track 15.7 -> 53.8 mm
- net /SIG_FRONT: track 15.7 -> 53.8 mm
- net /IR_1: track 87.4 -> 123.8 mm
- net /IR_12: track 115.0 -> 80.5 mm
- net /SCL: track 18.5 -> 52.6 mm, vias 0 -> 1
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- added copper zone on In1.Cu, net /VIN
Other:
- outline, holes or cut-outs redrawn
- board text added: "."
- board text added: "pull me down"
- board text added: "software is easy when you have good hardware, it's a shame I always fuck up on hardware"
- board text removed: "debugability they called it, fuckupability is better"
