File: BUCKY_MAIN/BUCKY_MAIN.kicad_sch (KiCad schematic)
At the start: 42 parts, among them J1 Conn_01x10, J2 Conn_01x06, J4 Conn_01x06

Commit message: fix: BUCKY_MAIN v2?
Parts:
- removed D14: D, Diode_SMD:D_0805_2012Metric, symbol Device:D
- added J3: Conn_01x01, Connector_PinHeader_2.54mm:PinHeader_1x01_P2.54mm_Vertical, symbol Connector_Generic:Conn_01x01
- D13: footprint Diode_SMD:D_0805_2012Metric -> Diode_SMD:D_3220_8050Metric
Connections:
- net +3.3V: now also D1.2 (A), D10.2 (A), D11.2 (A), D12.2 (A), D2.2 (A), D3.2 (A), D4.2 (A), D5.2 (A), D6.2 (A), D7.2 (A), D8.2 (A), D9.2 (A)
- net +5V: no longer A1.AREF, D1.2 (A), D10.2 (A), D11.2 (A), D12.2 (A), D2.2 (A), D3.2 (A), D4.2 (A), D5.2 (A), D6.2 (A), D7.2 (A), D8.2 (A), D9.2 (A)
- net IR_10: now also A1.41; no longer A1.13
- net IR_11: now also A1.49; no longer A1.52
- net IR_12: now also A1.51; no longer A1.53
- net IR_2: now also A1.53; no longer A1.51
- net IR_3: now also A1.52; no longer A1.48
- net IR_4: now also A1.11; no longer A1.43
- net IR_5: now also A1.13; no longer A1.23
- net IR_6: now also A1.12; no longer A1.17
- net IR_7: now also A1.4; no longer A1.5
- net IR_8: now also A1.5; no longer A1.11
- net IR_9: now also A1.17; no longer A1.12
- net M1_PWM: now also A1.8; no longer A1.2
- net M2_PWM: now also A1.9; no longer A1.3
- net M3_PWM: now also A1.10; no longer A1.4
- net SIG_BACK: now also A1.2; no longer A1.20
- net SIG_FRONT: now also A1.3; no longer A1.21
- net SIG_LEFT: now also A1.18; no longer A1.19
- net SIG_RIGHT: now also A1.19; no longer A1.18
- net VIN: now also J2.1 (Pin_1); no longer A1.VIN
- net RX0: now reaches A1.0
- net TX0: now reaches A1.1
- net D25: now reaches A1.25
- net D26: now reaches A1.26
- net D27: now reaches A1.27
- net D28: now reaches A1.28
- net D29: now reaches A1.29
- net D30: now reaches A1.30
- net D31: now reaches A1.31
- net D32: now reaches A1.32
- net D33: now reaches A1.33
- net D34: now reaches A1.34
- net D35: now reaches A1.35
- net D36: now reaches A1.36
- net D37: now reaches A1.37
- net D38: now reaches A1.38
- net D39: now reaches A1.39
- net D40: now reaches A1.40
- net D42: now reaches A1.42
- net D44: now reaches A1.44
- net D45: now reaches A1.45
- net D46: now reaches A1.46
- net D47: now reaches A1.47
- net D6: now reaches A1.6
- net D7: now reaches A1.7
- net A10: now reaches A1.AD10
- net A11: now reaches A1.AD11
- net A12: now reaches A1.AD12
- net A13: now reaches A1.AD13
- net A14: now reaches A1.AD14
- net A15: now reaches A1.AD15
- net A4: now reaches A1.AD4
- net A5: now reaches A1.AD5
- net A6: now reaches A1.AD6
- net A7: now reaches A1.AD7
- net A8: now reaches A1.AD8
- net A9: now reaches A1.AD9
- new net D20/SDA: A1.20
- new net D21/SCL: A1.21
- new net D23: A1.23
- new net D43: A1.43
- new net D48: A1.48
- new net VIN_12V: A1.VIN, J3.1 (Pin_1)
- no-connect marks 47 -> 6
Other:
- note added: "INT4"
- note added: "INT5"
- note removed: "INT0"
- note removed: "INT1"
